Commit message: Improve velocity tracking and add SLAM/Nav2 config
- Fix velocity tracking: add continuous cmd_vel publishing (10Hz) to
  prevent diff_drive_controller timeout (was causing 15% efficiency)
- Add laser_frame to URDF for Nav2 lidar integration
- Add lidar rangefinder sensors to MuJoCo model (8 beams at 45° intervals)
- Configure SLAM Toolbox parameters in nav2_params.yaml
- Increase motor torque (gear=500) and acceleration limits for responsive control
- Fix docker-compose volume mount to not overwrite mujoco_ros2_control
- Fix caster wheel positions to properly touch ground

🤖 Generated with [Claude Code](https://claude.com/claude-code)

Co-Authored-By: Claude <noreply@anthropic.com>

File: ros2_ws/src/sitebot_ros/urdf/sitebot.urdf.xacro (robot description, xacro)
@@ -66,4 +66,20 @@
     <origin xyz="0 0 0.32" rpy="0 0 0"/>
   </joint>
+  <!-- Laser/Lidar frame for Nav2 -->
+  <link name="laser_frame">
+    <visual>
+      <geometry>
+        <cylinder radius="0.04" length="0.02"/>
+      </geometry>
+      <material name="red">
+        <color rgba="0.8 0.1 0.1 1"/>
+      </material>
+    </visual>
+  </link>
+  <joint name="laser_joint" type="fixed">
+    <parent link="base_link"/>
+    <child link="laser_frame"/>
+    <origin xyz="0 0 0.30" rpy="0 0 0"/>
+  </joint>
   <!-- Left wheel -->
   <link name="left_wheel">
@@ -139,5 +155,5 @@
     <parent link="base_link"/>
     <child link="front_caster"/>
-    <origin xyz="0.35 0 -0.05" rpy="0 0 0"/>
+    <origin xyz="0.35 0 -0.10" rpy="0 0 0"/>
   </joint>
   <!-- Rear caster -->
@@ -162,5 +178,5 @@
     <parent link="base_link"/>
     <child link="rear_caster"/>
-    <origin xyz="-0.35 0 -0.05" rpy="0 0 0"/>
+    <origin xyz="-0.35 0 -0.10" rpy="0 0 0"/>
   </joint>
   <!-- ros2_control hardware interface -->
@@ -175,7 +191,4 @@
         <param name="max">20</param>
       </command_interface>
-      <param name="velocity_kp">50.0</param>
-      <param name="velocity_ki">5.0</param>
-      <param name="velocity_kd">0.1</param>
       <state_interface name="position"/>
       <state_interface name="velocity"/>
@@ -186,7 +199,4 @@
         <param name="max">20</param>
       </command_interface>
-      <param name="velocity_kp">50.0</param>
-      <param name="velocity_ki">5.0</param>
-      <param name="velocity_kd">0.1</param>
       <state_interface name="position"/>
       <state_interface name="velocity"/>
